File: Shield/capteur_graphite_arduino.kicad_sch (KiCad schematic)
At the start: 20 parts, among them J1 Power, J2 Digital/PWM, J3 Analog, J4 Digital/PWM, J5 Conn_01x02, U1 LTC1050, U3 encodeur_Rota, U5 U3 Bluetooth

Commit message: R_flex_sensor
Parts:
- R6: value 47k -> 33K
Changed lines of the file:
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@@
 			)
 		)
-		(property "Value" "47k"
+		(property "Value" "33K"
 			(at 240.03 137.1599 0)
 			(effects
